Commit message: add urdf and change tf

File: system_descriptor/urdf/arena_octagon.urdf (robot description, URDF)
Before this commit: robot arena_octagon, 85 links, 84 joints
Links:
- removed link odom
- added link CAP_L_6_link; collision box size=0.01 0.18250 0.233; visual box size=0.01 0.18250 0.233
- added link CAP_L_7_link; collision box size=0.01 0.18250 0.233; visual box size=0.01 0.18250 0.233
- added link CAP_L_WU_6_link; collision box size=0.01 0.12323 0.233; visual box size=0.01 0.12323 0.233
- added link CAP_L_WU_7_link; collision box size=0.01 0.12323 0.233; visual box size=0.01 0.12323 0.233
- added link CAP_R_6_link; collision box size=0.01 0.18250 0.233; visual box size=0.01 0.18250 0.233
- added link CAP_R_7_link; collision box size=0.01 0.18250 0.233; visual box size=0.01 0.18250 0.233
- added link CAP_R_WD_6_link; collision box size=0.01 0.12323 0.233; visual box size=0.01 0.12323 0.233
- added link CAP_R_WD_7_link; collision box size=0.01 0.12323 0.233; visual box size=0.01 0.12323 0.233
- added link TAM_0_6_link; collision box size=0.01 0.13917 0.233; visual box size=0.01 0.13917 0.233
- added link TAM_0_7_link; collision box size=0.01 0.13917 0.233; visual box size=0.01 0.13917 0.233
- added link TAM_0_WD_6_link; collision box size=0.01 0.12323 0.233; visual box size=0.01 0.12323 0.233
- added link TAM_0_WD_7_link; collision box size=0.01 0.12323 0.233; visual box size=0.01 0.12323 0.233
- added link TAM_0_WU_6_link; collision box size=0.01 0.12323 0.233; visual box size=0.01 0.12323 0.233
- added link TAM_0_WU_7_link; collision box size=0.01 0.12323 0.233; visual box size=0.01 0.12323 0.233
- added link TAM_1_6_link; collision box size=0.01 0.13917 0.233; visual box size=0.01 0.13917 0.233
- added link TAM_1_7_link; collision box size=0.01 0.13917 0.233; visual box size=0.01 0.13917 0.233
- added link TAM_1_WD_6_link; collision box size=0.01 0.12323 0.233; visual box size=0.01 0.12323 0.233
- added link TAM_1_WD_7_link; collision box size=0.01 0.12323 0.233; visual box size=0.01 0.12323 0.233
- added link TAM_1_WU_6_link; collision box size=0.01 0.12323 0.233; visual box size=0.01 0.12323 0.233
- added link TAM_1_WU_7_link; collision box size=0.01 0.12323 0.233; visual box size=0.01 0.12323 0.233
- added link TAM_2_6_link; collision box size=0.01 0.13917 0.233; visual box size=0.01 0.13917 0.233
- added link TAM_2_7_link; collision box size=0.01 0.13917 0.233; visual box size=0.01 0.13917 0.233
- added link TAM_2_WD_6_link; collision box size=0.01 0.12323 0.233; visual box size=0.01 0.12323 0.233
- added link TAM_2_WD_7_link; collision box size=0.01 0.12323 0.233; visual box size=0.01 0.12323 0.233
- added link TAM_2_WU_6_link; collision box size=0.01 0.12323 0.233; visual box size=0.01 0.12323 0.233
- added link TAM_2_WU_7_link; collision box size=0.01 0.12323 0.233; visual box size=0.01 0.12323 0.233
- added link WALL_6_link; collision box size=0.01 0.85328 0.233; visual box size=0.01 0.85328 0.233
- added link WALL_7_link; collision box size=0.01 0.85328 0.233; visual box size=0.01 0.85328 0.233
- added link center_camera
- link CAP_L_0_link: geometry collision box size=0.01 0.18250 0.233; visual box size=0.01 0.18250 0.233
- link CAP_L_1_link: geometry collision box size=0.01 0.18250 0.233; visual box size=0.01 0.18250 0.233
- link CAP_L_2_link: geometry collision box size=0.01 0.18250 0.233; visual box size=0.01 0.18250 0.233
- link CAP_L_3_link: geometry collision box size=0.01 0.18250 0.233; visual box size=0.01 0.18250 0.233
- link CAP_L_4_link: geometry collision box size=0.01 0.18250 0.233; visual box size=0.01 0.18250 0.233
- link CAP_L_5_link: geometry collision box size=0.01 0.18250 0.233; visual box size=0.01 0.18250 0.233
- link CAP_L_WU_0_link: geometry collision box size=0.01 0.12323 0.233; visual box size=0.01 0.12323 0.233
- link CAP_L_WU_1_link: geometry collision box size=0.01 0.12323 0.233; visual box size=0.01 0.12323 0.233
- link CAP_L_WU_2_link: geometry collision box size=0.01 0.12323 0.233; visual box size=0.01 0.12323 0.233
- link CAP_L_WU_3_link: geometry collision box size=0.01 0.12323 0.233; visual box size=0.01 0.12323 0.233
- link CAP_L_WU_4_link: geometry collision box size=0.01 0.12323 0.233; visual box size=0.01 0.12323 0.233
- link CAP_L_WU_5_link: geometry collision box size=0.01 0.12323 0.233; visual box size=0.01 0.12323 0.233
- link CAP_R_0_link: geometry collision box size=0.01 0.18250 0.233; visual box size=0.01 0.18250 0.233
- link CAP_R_1_link: geometry collision box size=0.01 0.18250 0.233; visual box size=0.01 0.18250 0.233
- link CAP_R_2_link: geometry collision box size=0.01 0.18250 0.233; visual box size=0.01 0.18250 0.233
- link CAP_R_3_link: geometry collision box size=0.01 0.18250 0.233; visual box size=0.01 0.18250 0.233
- link CAP_R_4_link: geometry collision box size=0.01 0.18250 0.233; visual box size=0.01 0.18250 0.233
- link CAP_R_5_link: geometry collision box size=0.01 0.18250 0.233; visual box size=0.01 0.18250 0.233
- link CAP_R_WD_0_link: geometry collision box size=0.01 0.12323 0.233; visual box size=0.01 0.12323 0.233
- link CAP_R_WD_1_link: geometry collision box size=0.01 0.12323 0.233; visual box size=0.01 0.12323 0.233
- link CAP_R_WD_2_link: geometry collision box size=0.01 0.12323 0.233; visual box size=0.01 0.12323 0.233
- link CAP_R_WD_3_link: geometry collision box size=0.01 0.12323 0.233; visual box size=0.01 0.12323 0.233
- link CAP_R_WD_4_link: geometry collision box size=0.01 0.12323 0.233; visual box size=0.01 0.12323 0.233
- link CAP_R_WD_5_link: geometry collision box size=0.01 0.12323 0.233; visual box size=0.01 0.12323 0.233
- link TAM_0_0_link: geometry collision box size=0.01 0.13917 0.233; visual box size=0.01 0.13917 0.233
- link TAM_0_1_link: geometry collision box size=0.01 0.13917 0.233; visual box size=0.01 0.13917 0.233
- link TAM_0_2_link: geometry collision box size=0.01 0.13917 0.233; visual box size=0.01 0.13917 0.233
- link TAM_0_3_link: geometry collision box size=0.01 0.13917 0.233; visual box size=0.01 0.13917 0.233
- link TAM_0_4_link: geometry collision box size=0.01 0.13917 0.233; visual box size=0.01 0.13917 0.233
- link TAM_0_5_link: geometry collision box size=0.01 0.13917 0.233; visual box size=0.01 0.13917 0.233
- link TAM_0_WD_0_link: geometry collision box size=0.01 0.12323 0.233; visual box size=0.01 0.12323 0.233
- link TAM_0_WD_1_link: geometry collision box size=0.01 0.12323 0.233; visual box size=0.01 0.12323 0.233
- link TAM_0_WD_2_link: geometry collision box size=0.01 0.12323 0.233; visual box size=0.01 0.12323 0.233
- link TAM_0_WD_3_link: geometry collision box size=0.01 0.12323 0.233; visual box size=0.01 0.12323 0.233
- link TAM_0_WD_4_link: geometry collision box size=0.01 0.12323 0.233; visual box size=0.01 0.12323 0.233
- link TAM_0_WD_5_link: geometry collision box size=0.01 0.12323 0.233; visual box size=0.01 0.12323 0.233
- link TAM_0_WU_0_link: geometry collision box size=0.01 0.12323 0.233; visual box size=0.01 0.12323 0.233
- link TAM_0_WU_1_link: geometry collision box size=0.01 0.12323 0.233; visual box size=0.01 0.12323 0.233
- link TAM_0_WU_2_link: geometry collision box size=0.01 0.12323 0.233; visual box size=0.01 0.12323 0.233
- link TAM_0_WU_3_link: geometry collision box size=0.01 0.12323 0.233; visual box size=0.01 0.12323 0.233
- link TAM_0_WU_4_link: geometry collision box size=0.01 0.12323 0.233; visual box size=0.01 0.12323 0.233
- link TAM_0_WU_5_link: geometry collision box size=0.01 0.12323 0.233; visual box size=0.01 0.12323 0.233
- link TAM_1_0_link: geometry collision box size=0.01 0.13917 0.233; visual box size=0.01 0.13917 0.233
- link TAM_1_1_link: geometry collision box size=0.01 0.13917 0.233; visual box size=0.01 0.13917 0.233
- link TAM_1_2_link: geometry collision box size=0.01 0.13917 0.233; visual box size=0.01 0.13917 0.233
- link TAM_1_3_link: geometry collision box size=0.01 0.13917 0.233; visual box size=0.01 0.13917 0.233
- link TAM_1_4_link: geometry collision box size=0.01 0.13917 0.233; visual box size=0.01 0.13917 0.233
- link TAM_1_5_link: geometry collision box size=0.01 0.13917 0.233; visual box size=0.01 0.13917 0.233
- link TAM_1_WD_0_link: geometry collision box size=0.01 0.12323 0.233; visual box size=0.01 0.12323 0.233
- link TAM_1_WD_1_link: geometry collision box size=0.01 0.12323 0.233; visual box size=0.01 0.12323 0.233
- link TAM_1_WD_2_link: geometry collision box size=0.01 0.12323 0.233; visual box size=0.01 0.12323 0.233
- link TAM_1_WD_3_link: geometry collision box size=0.01 0.12323 0.233; visual box size=0.01 0.12323 0.233
- link TAM_1_WD_4_link: geometry collision box size=0.01 0.12323 0.233; visual box size=0.01 0.12323 0.233
- link TAM_1_WD_5_link: geometry collision box size=0.01 0.12323 0.233; visual box size=0.01 0.12323 0.233
- link TAM_1_WU_0_link: geometry collision box size=0.01 0.12323 0.233; visual box size=0.01 0.12323 0.233
- link TAM_1_WU_1_link: geometry collision box size=0.01 0.12323 0.233; visual box size=0.01 0.12323 0.233
- link TAM_1_WU_2_link: geometry collision box size=0.01 0.12323 0.233; visual box size=0.01 0.12323 0.233
- link TAM_1_WU_3_link: geometry collision box size=0.01 0.12323 0.233; visual box size=0.01 0.12323 0.233
- link TAM_1_WU_4_link: geometry collision box size=0.01 0.12323 0.233; visual box size=0.01 0.12323 0.233
- link TAM_1_WU_5_link: geometry collision box size=0.01 0.12323 0.233; visual box size=0.01 0.12323 0.233
- link TAM_2_0_link: geometry collision box size=0.01 0.13917 0.233; visual box size=0.01 0.13917 0.233
- link TAM_2_1_link: geometry collision box size=0.01 0.13917 0.233; visual box size=0.01 0.13917 0.233
- link TAM_2_2_link: geometry collision box size=0.01 0.13917 0.233; visual box size=0.01 0.13917 0.233
- link TAM_2_3_link: geometry collision box size=0.01 0.13917 0.233; visual box size=0.01 0.13917 0.233
- link TAM_2_4_link: geometry collision box size=0.01 0.13917 0.233; visual box size=0.01 0.13917 0.233
- link TAM_2_5_link: geometry collision box size=0.01 0.13917 0.233; visual box size=0.01 0.13917 0.233
- link TAM_2_WD_0_link: geometry collision box size=0.01 0.12323 0.233; visual box size=0.01 0.12323 0.233
- link TAM_2_WD_1_link: geometry collision box size=0.01 0.12323 0.233; visual box size=0.01 0.12323 0.233
- link TAM_2_WD_2_link: geometry collision box size=0.01 0.12323 0.233; visual box size=0.01 0.12323 0.233
- link TAM_2_WD_3_link: geometry collision box size=0.01 0.12323 0.233; visual box size=0.01 0.12323 0.233
- link TAM_2_WD_4_link: geometry collision box size=0.01 0.12323 0.233; visual box size=0.01 0.12323 0.233
- link TAM_2_WD_5_link: geometry collision box size=0.01 0.12323 0.233; visual box size=0.01 0.12323 0.233
- link TAM_2_WU_0_link: geometry collision box size=0.01 0.12323 0.233; visual box size=0.01 0.12323 0.233
- link TAM_2_WU_1_link: geometry collision box size=0.01 0.12323 0.233; visual box size=0.01 0.12323 0.233
- link TAM_2_WU_2_link: geometry collision box size=0.01 0.12323 0.233; visual box size=0.01 0.12323 0.233
- link TAM_2_WU_3_link: geometry collision box size=0.01 0.12323 0.233; visual box size=0.01 0.12323 0.233
- link TAM_2_WU_4_link: geometry collision box size=0.01 0.12323 0.233; visual box size=0.01 0.12323 0.233
- link TAM_2_WU_5_link: geometry collision box size=0.01 0.12323 0.233; visual box size=0.01 0.12323 0.233
- link WALL_0_link: geometry collision box size=0.01 0.85328 0.233; visual box size=0.01 0.85328 0.233
- link WALL_1_link: geometry collision box size=0.01 0.85328 0.233; visual box size=0.01 0.85328 0.233
- link WALL_2_link: geometry collision box size=0.01 0.85328 0.233; visual box size=0.01 0.85328 0.233
- link WALL_3_link: geometry collision box size=0.01 0.85328 0.233; visual box size=0.01 0.85328 0.233
- link WALL_4_link: geometry collision box size=0.01 0.85328 0.233; visual box size=0.01 0.85328 0.233
- link WALL_5_link: geometry collision box size=0.01 0.85328 0.233; visual box size=0.01 0.85328 0.233
Joints:
- added joint CAP_L_6_joint: type fixed, parent center_camera, child CAP_L_6_link, origin xyz=-0.45736 -0.86441 0.11650 rpy=0 0 6.28319
- added joint CAP_L_7_joint: type fixed, parent center_camera, child CAP_L_7_link, origin xyz=0.28783 -0.93463 0.11650 rpy=0 0 7.06858
- added joint CAP_L_WU_6_joint: type fixed, parent center_camera, child CAP_L_WU_6_link, origin xyz=-0.42137 -0.98439 0.11650 rpy=0 0 7.06858
- added joint CAP_L_WU_7_joint: type fixed, parent center_camera, child CAP_L_WU_7_link, origin xyz=0.39812 -0.99402 0.11650 rpy=0 0 7.85398
- added joint CAP_R_6_joint: type fixed, parent center_camera, child CAP_R_6_link, origin xyz=0.45736 -0.86441 0.11650 rpy=0 0 6.28319
- added joint CAP_R_7_joint: type fixed, parent center_camera, child CAP_R_7_link, origin xyz=0.93463 -0.28783 0.11650 rpy=0 0 7.06858
- added joint CAP_R_WD_6_joint: type fixed, parent center_camera, child CAP_R_WD_6_link, origin xyz=0.42137 -0.98439 0.11650 rpy=0 0 5.49779
- added joint CAP_R_WD_7_joint: type fixed, parent center_camera, child CAP_R_WD_7_link, origin xyz=0.99402 -0.39812 0.11650 rpy=0 0 6.28319
- added joint TAM_0_6_joint: type fixed, parent center_camera, child TAM_0_6_link, origin xyz=-0.22496 -0.89440 0.11650 rpy=0 0 6.28319
- added joint TAM_0_7_joint: type fixed, parent center_camera, child TAM_0_7_link, origin xyz=0.47337 -0.79151 0.11650 rpy=0 0 7.06858
- added joint TAM_0_WD_6_joint: type fixed, parent center_camera, child TAM_0_WD_6_link, origin xyz=-0.18897 -0.98439 0.11650 rpy=0 0 7.06858
- added joint TAM_0_WD_7_joint: type fixed, parent center_camera, child TAM_0_WD_7_link, origin xyz=0.56245 -0.82969 0.11650 rpy=0 0 7.85398
- added joint TAM_0_WU_6_joint: type fixed, parent center_camera, child TAM_0_WU_6_link, origin xyz=-0.26095 -0.98439 0.11650 rpy=0 0 5.49779
- added joint TAM_0_WU_7_joint: type fixed, parent center_camera, child TAM_0_WU_7_link, origin xyz=0.51155 -0.88059 0.11650 rpy=0 0 6.28319
- added joint TAM_1_6_joint: type fixed, parent center_camera, child TAM_1_6_link, origin xyz=-0.00000 -0.89440 0.11650 rpy=0 0 6.28319
- added joint TAM_1_7_joint: type fixed, parent center_camera, child TAM_1_7_link, origin xyz=0.63244 -0.63244 0.11650 rpy=0 0 7.06858
- added joint TAM_1_WD_6_joint: type fixed, parent center_camera, child TAM_1_WD_6_link, origin xyz=0.03599 -0.98439 0.11650 rpy=0 0 7.06858
- added joint TAM_1_WD_7_joint: type fixed, parent center_camera, child TAM_1_WD_7_link, origin xyz=0.72152 -0.67062 0.11650 rpy=0 0 7.85398
- added joint TAM_1_WU_6_joint: type fixed, parent center_camera, child TAM_1_WU_6_link, origin xyz=-0.03599 -0.98439 0.11650 rpy=0 0 5.49779
- added joint TAM_1_WU_7_joint: type fixed, parent center_camera, child TAM_1_WU_7_link, origin xyz=0.67062 -0.72152 0.11650 rpy=0 0 6.28319
- added joint TAM_2_6_joint: type fixed, parent center_camera, child TAM_2_6_link, origin xyz=0.22496 -0.89440 0.11650 rpy=0 0 6.28319
- added joint TAM_2_7_joint: type fixed, parent center_camera, child TAM_2_7_link, origin xyz=0.79151 -0.47337 0.11650 rpy=0 0 7.06858
- added joint TAM_2_WD_6_joint: type fixed, parent center_camera, child TAM_2_WD_6_link, origin xyz=0.26095 -0.98439 0.11650 rpy=0 0 7.06858
- added joint TAM_2_WD_7_joint: type fixed, parent center_camera, child TAM_2_WD_7_link, origin xyz=0.88059 -0.51155 0.11650 rpy=0 0 7.85398
- added joint TAM_2_WU_6_joint: type fixed, parent center_camera, child TAM_2_WU_6_link, origin xyz=0.18897 -0.98439 0.11650 rpy=0 0 5.49779
- added joint TAM_2_WU_7_joint: type fixed, parent center_camera, child TAM_2_WU_7_link, origin xyz=0.82969 -0.56245 0.11650 rpy=0 0 6.28319
- added joint WALL_6_joint: type fixed, parent center_camera, child WALL_6_link, origin xyz=-0.00000 -1.03000 0.11650 rpy=0 0 4.71239
- added joint WALL_7_joint: type fixed, parent center_camera, child WALL_7_link, origin xyz=0.72832 -0.72832 0.11650 rpy=0 0 5.49779
- joint CAP_L_0_joint: parent odom -> center_camera
- joint CAP_L_1_joint: origin xyz=0.82828 0.51992 0.11650 rpy=0 0 2.61799 -> xyz=0.93463 0.28783 0.11650 rpy=0 0 2.35619; parent odom -> center_camera
- joint CAP_L_2_joint: origin xyz=-0.03612 0.97728 0.11650 rpy=0 0 3.66519 -> xyz=0.45736 0.86441 0.11650 rpy=0 0 3.14159; parent odom -> center_camera
- joint CAP_L_3_joint: origin xyz=-0.86441 0.45736 0.11650 rpy=0 0 4.71239 -> xyz=-0.28783 0.93463 0.11650 rpy=0 0 3.92699; parent odom -> center_camera
- joint CAP_L_4_joint: origin xyz=-0.82828 -0.51992 0.11650 rpy=0 0 5.75959 -> xyz=-0.86441 0.45736 0.11650 rpy=0 0 4.71239; parent odom -> center_camera
- joint CAP_L_5_joint: origin xyz=0.03612 -0.97728 0.11650 rpy=0 0 0.52360 -> xyz=-0.93463 -0.28783 0.11650 rpy=0 0 5.49779; parent odom -> center_camera
- joint CAP_L_WU_0_joint: parent odom -> center_camera
- joint CAP_L_WU_1_joint: origin xyz=0.85711 0.64182 0.11650 rpy=0 0 3.40339 -> xyz=0.99402 0.39812 0.11650 rpy=0 0 3.14159; parent odom -> center_camera
- joint CAP_L_WU_2_joint: origin xyz=-0.12728 1.06319 0.11650 rpy=0 0 4.45059 -> xyz=0.42137 0.98439 0.11650 rpy=0 0 3.92699; parent odom -> center_camera
- joint CAP_L_WU_3_joint: origin xyz=-0.98439 0.42137 0.11650 rpy=0 0 5.49779 -> xyz=-0.39812 0.99402 0.11650 rpy=0 0 4.71239; parent odom -> center_camera
- joint CAP_L_WU_4_joint: origin xyz=-0.85711 -0.64182 0.11650 rpy=0 0 0.26180 -> xyz=-0.98439 0.42137 0.11650 rpy=0 0 5.49779; parent odom -> center_camera
- joint CAP_L_WU_5_joint: origin xyz=0.12728 -1.06319 0.11650 rpy=0 0 1.30900 -> xyz=-0.99402 -0.39812 0.11650 rpy=0 0 6.28319; parent odom -> center_camera
- joint CAP_R_0_joint: parent odom -> center_camera
- joint CAP_R_1_joint: origin xyz=0.03612 0.97728 0.11650 rpy=0 0 2.61799 -> xyz=0.28783 0.93463 0.11650 rpy=0 0 2.35619; parent odom -> center_camera
- joint CAP_R_2_joint: origin xyz=-0.82828 0.51992 0.11650 rpy=0 0 3.66519 -> xyz=-0.45736 0.86441 0.11650 rpy=0 0 3.14159; parent odom -> center_camera
- joint CAP_R_3_joint: origin xyz=-0.86441 -0.45736 0.11650 rpy=0 0 4.71239 -> xyz=-0.93463 0.28783 0.11650 rpy=0 0 3.92699; parent odom -> center_camera
- joint CAP_R_4_joint: origin xyz=-0.03612 -0.97728 0.11650 rpy=0 0 5.75959 -> xyz=-0.86441 -0.45736 0.11650 rpy=0 0 4.71239; parent odom -> center_camera
- joint CAP_R_5_joint: origin xyz=0.82828 -0.51992 0.11650 rpy=0 0 0.52360 -> xyz=-0.28783 -0.93463 0.11650 rpy=0 0 5.49779; parent odom -> center_camera
- joint CAP_R_WD_0_joint: parent odom -> center_camera
- joint CAP_R_WD_1_joint: origin xyz=0.12728 1.06319 0.11650 rpy=0 0 1.83260 -> xyz=0.39812 0.99402 0.11650 rpy=0 0 1.57080; parent odom -> center_camera
- joint CAP_R_WD_2_joint: origin xyz=-0.85711 0.64182 0.11650 rpy=0 0 2.87979 -> xyz=-0.42137 0.98439 0.11650 rpy=0 0 2.35619; parent odom -> center_camera
- joint CAP_R_WD_3_joint: origin xyz=-0.98439 -0.42137 0.11650 rpy=0 0 3.92699 -> xyz=-0.99402 0.39812 0.11650 rpy=0 0 3.14159; parent odom -> center_camera
- joint CAP_R_WD_4_joint: origin xyz=-0.12728 -1.06319 0.11650 rpy=0 0 4.97419 -> xyz=-0.98439 -0.42137 0.11650 rpy=0 0 3.92699; parent odom -> center_camera
- joint CAP_R_WD_5_joint: origin xyz=0.85711 -0.64182 0.11650 rpy=0 0 6.02139 -> xyz=-0.39812 -0.99402 0.11650 rpy=0 0 4.71239; parent odom -> center_camera
- joint TAM_0_0_joint: parent odom -> center_camera
- joint TAM_0_1_joint: origin xyz=0.64203 0.66209 0.11650 rpy=0 0 2.61799 -> xyz=0.79151 0.47337 0.11650 rpy=0 0 2.35619; parent odom -> center_camera
- joint TAM_0_2_joint: origin xyz=-0.25238 0.88705 0.11650 rpy=0 0 3.66519 -> xyz=0.22496 0.89440 0.11650 rpy=0 0 3.14159; parent odom -> center_camera
- joint TAM_0_3_joint: origin xyz=-0.89440 0.22496 0.11650 rpy=0 0 4.71239 -> xyz=-0.47337 0.79151 0.11650 rpy=0 0 3.92699; parent odom -> center_camera
- joint TAM_0_4_joint: origin xyz=-0.64203 -0.66209 0.11650 rpy=0 0 5.75959 -> xyz=-0.89440 0.22496 0.11650 rpy=0 0 4.71239; parent odom -> center_camera
- joint TAM_0_5_joint: origin xyz=0.25238 -0.88705 0.11650 rpy=0 0 0.52360 -> xyz=-0.79151 -0.47337 0.11650 rpy=0 0 5.49779; parent odom -> center_camera
- joint TAM_0_WD_0_joint: parent odom -> center_camera
- joint TAM_0_WD_1_joint: origin xyz=0.65584 0.75802 0.11650 rpy=0 0 3.40339 -> xyz=0.82969 0.56245 0.11650 rpy=0 0 3.14159; parent odom -> center_camera
- joint TAM_0_WD_2_joint: origin xyz=-0.32854 0.94699 0.11650 rpy=0 0 4.45059 -> xyz=0.18897 0.98439 0.11650 rpy=0 0 3.92699; parent odom -> center_camera
- joint TAM_0_WD_3_joint: origin xyz=-0.98439 0.18897 0.11650 rpy=0 0 5.49779 -> xyz=-0.56245 0.82969 0.11650 rpy=0 0 4.71239; parent odom -> center_camera
- joint TAM_0_WD_4_joint: origin xyz=-0.65584 -0.75802 0.11650 rpy=0 0 0.26180 -> xyz=-0.98439 0.18897 0.11650 rpy=0 0 5.49779; parent odom -> center_camera
- joint TAM_0_WD_5_joint: origin xyz=0.32854 -0.94699 0.11650 rpy=0 0 1.30900 -> xyz=-0.82969 -0.56245 0.11650 rpy=0 0 6.28319; parent odom -> center_camera
- joint TAM_0_WU_0_joint: parent odom -> center_camera
- joint TAM_0_WU_1_joint: origin xyz=0.71819 0.72203 0.11650 rpy=0 0 1.83260 -> xyz=0.88059 0.51155 0.11650 rpy=0 0 1.57080; parent odom -> center_camera
- joint TAM_0_WU_2_joint: origin xyz=-0.26620 0.98298 0.11650 rpy=0 0 2.87979 -> xyz=0.26095 0.98439 0.11650 rpy=0 0 2.35619; parent odom -> center_camera
- joint TAM_0_WU_3_joint: origin xyz=-0.98439 0.26095 0.11650 rpy=0 0 3.92699 -> xyz=-0.51155 0.88059 0.11650 rpy=0 0 3.14159; parent odom -> center_camera
- joint TAM_0_WU_4_joint: origin xyz=-0.71819 -0.72203 0.11650 rpy=0 0 4.97419 -> xyz=-0.98439 0.26095 0.11650 rpy=0 0 3.92699; parent odom -> center_camera
- joint TAM_0_WU_5_joint: origin xyz=0.26620 -0.98298 0.11650 rpy=0 0 6.02139 -> xyz=-0.88059 -0.51155 0.11650 rpy=0 0 4.71239; parent odom -> center_camera
- joint TAM_1_0_joint: parent odom -> center_camera
- joint TAM_1_1_joint: origin xyz=0.44720 0.77457 0.11650 rpy=0 0 2.61799 -> xyz=0.63244 0.63244 0.11650 rpy=0 0 2.35619; parent odom -> center_camera
- joint TAM_1_2_joint: origin xyz=-0.44720 0.77457 0.11650 rpy=0 0 3.66519 -> xyz=0.00000 0.89440 0.11650 rpy=0 0 3.14159; parent odom -> center_camera
- joint TAM_1_3_joint: origin xyz=-0.89440 0.00000 0.11650 rpy=0 0 4.71239 -> xyz=-0.63244 0.63244 0.11650 rpy=0 0 3.92699; parent odom -> center_camera
- joint TAM_1_4_joint: origin xyz=-0.44720 -0.77457 0.11650 rpy=0 0 5.75959 -> xyz=-0.89440 0.00000 0.11650 rpy=0 0 4.71239; parent odom -> center_camera
- joint TAM_1_5_joint: origin xyz=0.44720 -0.77457 0.11650 rpy=0 0 0.52360 -> xyz=-0.63244 -0.63244 0.11650 rpy=0 0 5.49779; parent odom -> center_camera
- joint TAM_1_WD_0_joint: parent odom -> center_camera
- joint TAM_1_WD_1_joint: origin xyz=0.46102 0.87050 0.11650 rpy=0 0 3.40339 -> xyz=0.67062 0.72152 0.11650 rpy=0 0 3.14159; parent odom -> center_camera
- joint TAM_1_WD_2_joint: origin xyz=-0.52336 0.83451 0.11650 rpy=0 0 4.45059 -> xyz=-0.03599 0.98439 0.11650 rpy=0 0 3.92699; parent odom -> center_camera
- joint TAM_1_WD_3_joint: origin xyz=-0.98439 -0.03599 0.11650 rpy=0 0 5.49779 -> xyz=-0.72152 0.67062 0.11650 rpy=0 0 4.71239; parent odom -> center_camera
- joint TAM_1_WD_4_joint: origin xyz=-0.46102 -0.87050 0.11650 rpy=0 0 0.26180 -> xyz=-0.98439 -0.03599 0.11650 rpy=0 0 5.49779; parent odom -> center_camera
- joint TAM_1_WD_5_joint: origin xyz=0.52336 -0.83451 0.11650 rpy=0 0 1.30900 -> xyz=-0.67062 -0.72152 0.11650 rpy=0 0 6.28319; parent odom -> center_camera
- joint TAM_1_WU_0_joint: parent odom -> center_camera
- joint TAM_1_WU_1_joint: origin xyz=0.52336 0.83451 0.11650 rpy=0 0 1.83260 -> xyz=0.72152 0.67062 0.11650 rpy=0 0 1.57080; parent odom -> center_camera
- joint TAM_1_WU_2_joint: origin xyz=-0.46102 0.87050 0.11650 rpy=0 0 2.87979 -> xyz=0.03599 0.98439 0.11650 rpy=0 0 2.35619; parent odom -> center_camera
- joint TAM_1_WU_3_joint: origin xyz=-0.98439 0.03599 0.11650 rpy=0 0 3.92699 -> xyz=-0.67062 0.72152 0.11650 rpy=0 0 3.14159; parent odom -> center_camera
- joint TAM_1_WU_4_joint: origin xyz=-0.52336 -0.83451 0.11650 rpy=0 0 4.97419 -> xyz=-0.98439 0.03599 0.11650 rpy=0 0 3.92699; parent odom -> center_camera
- joint TAM_1_WU_5_joint: origin xyz=0.46102 -0.87050 0.11650 rpy=0 0 6.02139 -> xyz=-0.72152 -0.67062 0.11650 rpy=0 0 4.71239; parent odom -> center_camera
- joint TAM_2_0_joint: parent odom -> center_camera
- joint TAM_2_1_joint: origin xyz=0.25238 0.88705 0.11650 rpy=0 0 2.61799 -> xyz=0.47337 0.79151 0.11650 rpy=0 0 2.35619; parent odom -> center_camera
- joint TAM_2_2_joint: origin xyz=-0.64203 0.66209 0.11650 rpy=0 0 3.66519 -> xyz=-0.22496 0.89440 0.11650 rpy=0 0 3.14159; parent odom -> center_camera
- joint TAM_2_3_joint: origin xyz=-0.89440 -0.22496 0.11650 rpy=0 0 4.71239 -> xyz=-0.79151 0.47337 0.11650 rpy=0 0 3.92699; parent odom -> center_camera
- joint TAM_2_4_joint: origin xyz=-0.25238 -0.88705 0.11650 rpy=0 0 5.75959 -> xyz=-0.89440 -0.22496 0.11650 rpy=0 0 4.71239; parent odom -> center_camera
- joint TAM_2_5_joint: origin xyz=0.64203 -0.66209 0.11650 rpy=0 0 0.52360 -> xyz=-0.47337 -0.79151 0.11650 rpy=0 0 5.49779; parent odom -> center_camera
- joint TAM_2_WD_0_joint: parent odom -> center_camera
- joint TAM_2_WD_1_joint: origin xyz=0.26620 0.98298 0.11650 rpy=0 0 3.40339 -> xyz=0.51155 0.88059 0.11650 rpy=0 0 3.14159; parent odom -> center_camera
- joint TAM_2_WD_2_joint: origin xyz=-0.71819 0.72203 0.11650 rpy=0 0 4.45059 -> xyz=-0.26095 0.98439 0.11650 rpy=0 0 3.92699; parent odom -> center_camera
- joint TAM_2_WD_3_joint: origin xyz=-0.98439 -0.26095 0.11650 rpy=0 0 5.49779 -> xyz=-0.88059 0.51155 0.11650 rpy=0 0 4.71239; parent odom -> center_camera
- joint TAM_2_WD_4_joint: origin xyz=-0.26620 -0.98298 0.11650 rpy=0 0 0.26180 -> xyz=-0.98439 -0.26095 0.11650 rpy=0 0 5.49779; parent odom -> center_camera
- joint TAM_2_WD_5_joint: origin xyz=0.71819 -0.72203 0.11650 rpy=0 0 1.30900 -> xyz=-0.51155 -0.88059 0.11650 rpy=0 0 6.28319; parent odom -> center_camera
- joint TAM_2_WU_0_joint: parent odom -> center_camera
- joint TAM_2_WU_1_joint: origin xyz=0.32854 0.94699 0.11650 rpy=0 0 1.83260 -> xyz=0.56245 0.82969 0.11650 rpy=0 0 1.57080; parent odom -> center_camera
- joint TAM_2_WU_2_joint: origin xyz=-0.65584 0.75802 0.11650 rpy=0 0 2.87979 -> xyz=-0.18897 0.98439 0.11650 rpy=0 0 2.35619; parent odom -> center_camera
- joint TAM_2_WU_3_joint: origin xyz=-0.98439 -0.18897 0.11650 rpy=0 0 3.92699 -> xyz=-0.82969 0.56245 0.11650 rpy=0 0 3.14159; parent odom -> center_camera
- joint TAM_2_WU_4_joint: origin xyz=-0.32854 -0.94699 0.11650 rpy=0 0 4.97419 -> xyz=-0.98439 -0.18897 0.11650 rpy=0 0 3.92699; parent odom -> center_camera
- joint TAM_2_WU_5_joint: origin xyz=0.65584 -0.75802 0.11650 rpy=0 0 6.02139 -> xyz=-0.56245 -0.82969 0.11650 rpy=0 0 4.71239; parent odom -> center_camera
- joint WALL_0_joint: parent odom -> center_camera
- joint WALL_1_joint: origin xyz=0.51500 0.89201 0.11650 rpy=0 0 1.04720 -> xyz=0.72832 0.72832 0.11650 rpy=0 0 0.78540; parent odom -> center_camera
- joint WALL_2_joint: origin xyz=-0.51500 0.89201 0.11650 rpy=0 0 2.09440 -> xyz=0.00000 1.03000 0.11650 rpy=0 0 1.57080; parent odom -> center_camera
- joint WALL_3_joint: origin xyz=-1.03000 0.00000 0.11650 rpy=0 0 3.14159 -> xyz=-0.72832 0.72832 0.11650 rpy=0 0 2.35619; parent odom -> center_camera
- joint WALL_4_joint: origin xyz=-0.51500 -0.89201 0.11650 rpy=0 0 4.18879 -> xyz=-1.03000 0.00000 0.11650 rpy=0 0 3.14159; parent odom -> center_camera
- joint WALL_5_joint: origin xyz=0.51500 -0.89201 0.11650 rpy=0 0 5.23599 -> xyz=-0.72832 -0.72832 0.11650 rpy=0 0 3.92699; parent odom -> center_camera
