Commit message: change all architecture

File: system_descriptor/urdf/base.xacro (robot description, xacro)
@@ -4,9 +4,9 @@
     <xacro:property name="base_scale" value="0.5 0.5 0.5" />
     <xacro:macro name="base">
-        <link name="base_link_3">
+        <link name="base_link_10">
             <visual>
                 <origin xyz="0 0 0" rpy="0 0 0" />
                 <geometry>
-                    <mesh filename="package://track_sys/meshes/qupa.dae" scale="${base_scale}" />
+                    <mesh filename="package://system_descriptor/meshes/qupa.dae" scale="${base_scale}" />
                 </geometry>
             </visual>

Commit message: make parametrization

File: system_descriptor/urdf/base.xacro (robot description, xacro)
@@ -1,8 +1,9 @@
 <?xml version="1.0"?>
 <robot xmlns:xacro="http://www.ros.org/wiki/xacro" name="epuck">
+    <xacro:arg name="id_robot" default=""/>
     <xacro:property name="base_mass" value="1" />
     <xacro:property name="base_scale" value="0.5 0.5 0.5" />
     <xacro:macro name="base">
-        <link name="base_link_10">
+        <link name="base_link_$(arg id_robot)">
             <visual>
                 <origin xyz="0 0 0" rpy="0 0 0" />

Commit message: add rosbag

File: system_descriptor/urdf/base.xacro (robot description, xacro)
@@ -3,5 +3,5 @@
     <xacro:arg name="id_robot" default=""/>
     <xacro:property name="base_mass" value="1" />
-    <xacro:property name="base_scale" value="0.5 0.5 0.5" />
+    <xacro:property name="base_scale" value="1 1 1" />
     <xacro:macro name="base">
         <link name="base_link_$(arg id_robot)">
